File: Schematic/PSU/PSU.sch (KiCad schematic (older format))
At the start: 34 parts, among them J1 Conn_01x01, J2 Conn_01x01, J3 Conn_01x06, T1 VPP24-210, U1 LM7812_TO220, U2 LM7912_TO220, U3 L78L05_SOT89, U4 B0505S-1W

Commit message: Added missing resistor: R15
Parts:
- F1: footprint myDevices:FuseHolder_5x20_Bare -> Fuse:Fuse_Littelfuse_372_D8.50mm
Changed lines of the file:
@@
 F 0 "F1" V 828 1625 50  0000 C CNN
 F 1 "T100mA" V 919 1625 50  0000 C CNN
-F 2 "myDevices:FuseHolder_5x20_Bare" V 955 1625 50  0001 C CNN
+F 2 "Fuse:Fuse_Littelfuse_372_D8.50mm" V 955 1625 50  0001 C CNN
 F 3 "~" H 1025 1625 50  0001 C CNN
 	1    1025 1625
